File: mspm0.kicad_pcb (KiCad board)
At the start: 4 copper layers, 66.8 x 85.8 mm, 128 parts, among them J1 Barrel_Jack_Switch_Pin3Ring, J10 USB_C_Receptacle_PowerOnly_6P, J11 Conn_01x04_MountingPin, J12 Conn_01x18_Pin, J2 Conn_01x02_Pin, J3 Conn_01x04_Pin, J4 Conn_01x04_Pin, J5 Conn_01x04_MountingPin, J6 Conn_01x04_Pin, J7 Conn_01x04_Pin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

Commit message: fixed floating bsl_pin
Parts:
- turned D1 to -90 degrees
Connections:
- D12 pad 2: /BOOT0 -> /BSL_invoke
- Q3 pad 2: /BOOT0 -> /BSL_invoke
- R37 pad 1: /BOOT0 -> /BSL_invoke
Routing:
- net /BSL_invoke: track 0.00 -> 38.2 mm, vias 0 -> 2
- net Net-(Q1-C): track 18.3 -> 21.9 mm
- net /BOOT0: track 3.23 -> 0.00 mm
- net Net-(D1-K): track 6.80 -> 3.88 mm
- net /PA16_A1_1: track 23.3 -> 25.6 mm
- net /PA15_A1_0: track 24.5 -> 26.3 mm
- net Net-(D13-K): track 12.3 -> 13.8 mm
- net /PA1: track 48.0 -> 49.3 mm
- net /PB17_A1_4: track 23.1 -> 21.8 mm
- net /PA8: track 46.0 -> 47.1 mm
- net /PA28: track 21.4 -> 22.5 mm
- net /PA14: track 22.9 -> 24.0 mm
- net /PA9: track 36.6 -> 37.6 mm
- net /PA10: track 65.9 -> 66.9 mm
- net /PA27_A0_0: track 16.1 -> 15.2 mm
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- added copper zone on F.Cu, net Net-(D1-K)

Commit message: updated silkscreen rev version number
Other:
- board text added: "Author: Alipay Date: 2024-07-16 Version:V1.2 MSPM0-DevBoard"
- board text removed: "Author: Alipay Date: 2024-04-16 Version:V1.1 MSPM0-DevBoard"
Changed lines of the file:
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@@
 		)
 	)
-	(gr_text "Author: Alipay\nDate:   2024-04-16\nVersion:V1.1\nMSPM0-DevBoard"
+	(gr_text "Author: Alipay\nDate:   2024-07-16\nVersion:V1.2\nMSPM0-DevBoard"
 		(at 181.35 40.15 0)
 		(layer "B.SilkS")
